Commit message: adjusted params

File: tuc_vehicle_description/urdf/vehicle.xacro (robot description, xacro)
@@ -2,11 +2,11 @@
 <robot xmlns:xacro="http://ros.org/wiki/xacro">
   <!-- load parameter -->
-  <xacro:property name="vehicle_info" value="${xacro.load_yaml('$(find sample_vehicle_description)/config/vehicle_info.param.yaml')}"/>
+  <xacro:property name="vehicle_info" value="${xacro.load_yaml('$(find tuc_vehicle_description)/config/vehicle_info.param.yaml')}"/>
   <!-- vehicle body -->
   <link name="base_link">
     <visual>
-      <origin xyz="${vehicle_info['/**']['ros__parameters']['wheel_base']/2.0} 0 0" rpy="${pi/2.0} 0 ${pi}"/>
+      <origin xyz="${vehicle_info['/**']['ros__parameters']['wheel_base']/2.0} 0 0" rpy="${pi/2.0} 0 0"/>
       <geometry>
-        <mesh filename="package://sample_vehicle_description/mesh/lexus.dae" scale="1 1 1"/>
+        <mesh filename="package://tuc_vehicle_description/mesh/volkswagen_id_buzz.fbx" scale="0.01 0.01 0.01"/>
       </geometry>
     </visual>

Commit message: fixed vehicle orientation

File: tuc_vehicle_description/urdf/vehicle.xacro (robot description, xacro)
@@ -6,5 +6,5 @@
   <link name="base_link">
     <visual>
-      <origin xyz="${vehicle_info['/**']['ros__parameters']['wheel_base']/2.0} 0 0" rpy="${pi/2.0} 0 0"/>
+      <origin xyz="${vehicle_info['/**']['ros__parameters']['wheel_base']/2.0} 0 0" rpy="0 0 ${pi/2.0}"/>
       <geometry>
         <mesh filename="package://tuc_vehicle_description/mesh/volkswagen_id_buzz.fbx" scale="0.01 0.01 0.01"/>

Commit message: fixed vehicle position

File: tuc_vehicle_description/urdf/vehicle.xacro (robot description, xacro)
@@ -6,5 +6,5 @@
   <link name="base_link">
     <visual>
-      <origin xyz="${vehicle_info['/**']['ros__parameters']['wheel_base']/2.0} 0 0" rpy="0 0 ${pi/2.0}"/>
+      <origin xyz="3.775 0 0" rpy="0 0 ${pi/2.0}"/>
       <geometry>
         <mesh filename="package://tuc_vehicle_description/mesh/volkswagen_id_buzz.fbx" scale="0.01 0.01 0.01"/>
